Commit message: pick place 2D camera simple

File: src/custom_robot_description/urdf/custom_gripper.xacro (robot description, xacro)
@@ -31,5 +31,5 @@
             <child link="finger_right"/>
             <axis xyz="1 0 0"/>
-            <limit lower="0" upper="0.044" velocity="0.5" effort="200"/>
+            <limit lower="0" upper="0.044" velocity="0.5" effort="400"/>
             <origin xyz="-0.05 0.0 0.011" rpy="0 0 0"/>
             <dynamics damping="1" friction="2"/>
@@ -42,7 +42,8 @@
             <child link="finger_left"/>
             <axis xyz="1 0 0"/>
-            <limit lower="-0.044" upper="0" velocity="0.5" effort="200"/>
+            <limit lower="-0.044" upper="0" velocity="0.5" effort="400"/>
             <origin xyz="0.05 0.0 0.011" rpy="0 0 0"/>
-            <dynamics damping="1" friction="2"/>
+            <!-- <dynamics damping="1" friction="2"/> -->
+            <dynamics friction="2"/>
             <mimic joint="finger_right_joint" multiplier="-1.0" offset="0" />
         </joint>
