Commit message: ur5 throubleshooting

File: src/ur5_description/urdf/ur5_gripper_camera.xacro (robot description, xacro)
@@ -14,9 +14,9 @@
         <parent link="world"/>
         <child link="base_link"/>
-        <origin xyz="0 0.0 0.8" rpy="0 0 0"/>
+        <origin xyz="0 0.0 0.8" rpy="0 0 -1.57"/>
   </joint>
   <!-- Define RGB-D sensor -->
   <xacro:kinetic_rgb name="rgbd_camera" parent="base">
-    <origin xyz="0.1 0.0 1.2" rpy="${0.0 * deg_to_rad} ${70.0 * deg_to_rad} ${0.0 * deg_to_rad}"/>
+    <origin xyz="0.1 0.0 1.2" rpy="${0.0 * deg_to_rad} ${70.0 * deg_to_rad} ${90 * deg_to_rad}"/>
     <origin xyz="0 0 0" rpy="${-90 * deg_to_rad} ${0 * deg_to_rad} ${-90 * deg_to_rad}" />
   </xacro:kinetic_rgb>
